File: 2_10decoder.sch (EAGLE design)
At the start: 255 parts, among them T1 BC847, T10 BC847, T11 BC847, T12 BC847, T13 BC847, T14 BC847, T15 BC847, T16 BC847, T17 BC847, T18 BC847, T19 BC847, T2 BC847, T20 BC847, T21 BC847, T22 BC847, T23 BC847, T24 BC847, T25 BC847, T26 BC847, T27 BC847, T28 BC847, T29 BC847, T3 BC847, T30 BC847, T31 BC847, T32 BC847, T33 BC847, T34 BC847, T35 BC847, T36 BC847, T37 BC847, T38 BC847, T39 BC847, T4 BC847, T40 BC847, T41 BC847, T42 BC847, T43 BC847, T44 BC847, T45 BC847, T46 BC847, T47 BC847, T48 BC847, T49 BC847, T5 BC847, T50 BC847, T51 BC847, T52 BC847, T53 BC847, T54 BC847, T55 BC847, T56 BC847, T57 BC847, T58 BC847, T59 BC847, T6 BC847, T60 BC847, T61 BC847, T62 BC847, T63 BC847, T64 BC847, T65 BC847, T66 BC847, T67 BC847, T68 BC847, T69 BC847, T7 BC847, T70 BC847, T8 BC847, T9 BC847

Commit message: 2_10 decoter second approach
Parts:
- removed LED13, LED14, LED15, LED16, LED17, LED18, LED19, LED20, LED21, LED22, LED23, LED24, LED25, LED26, LED27, LED28, LED29, LED30, LED31, LED32, LED33, LED34, LED35, LED36, LED37, LED38: (no value), led:LEDCHIP-LED0805
- removed R100, R101, R102, R103, R104, R105, R106, R107, R108, R109, R110, R111, R112, R113, R114, R115, R116, R117, R118, R119, R120, R121, R122, R123, R124, R125, R126, R127, R128, R129, R130, R131, R132, R133, R134, R135, R136, R137, R138, R139, R140, R141, R142, R143, R144, R145, R146, R53, R60, R61, R62, R63, R64, R65, R66, R67, R68, R69, R70, R71, R72, R73, R74, R75, R76, R77, R78, R79, R80, R81, R82, R83, R84, R85, R86, R87, R88, R89, R90, R91, R92, R93, R94, R95, R96, R97, R98, R99: (no value), resistor:R-EU_M0805
- removed T24, T26, T27, T28, T29, T30, T31, T32, T33, T34, T35, T36, T37, T38, T39, T40, T41, T42, T43, T44, T45, T46, T47, T48, T49, T50, T51, T52, T53, T54, T55, T56, T57, T58, T59, T60, T61, T62, T63, T64, T65, T66, T67, T68, T69, T70: BC847, transistor-neu-to92:BC847
- R1, R10, R2, R25, R26, R27, R28, R29, R3, R30, R31, R32, R33, R34, R4, R49, R5, R50, R51, R52, R6, R7, R8, R9: value (none) -> 10k
- R11, R13, R15, R17, R19, R35, R37, R39, R41, R43, R54, R56: value (none) -> 3K9
- R21, R22, R23, R24, R45, R46, R47, R48, R58, R59: device resistor:R-EU_M0805 -> rcl:R-EU_M1206
Connections:
- removed net N$100: LED24.A, R94.1
- removed net N$101: R95.1, T47.B
- removed net N$102: T48.E, T49.C
- removed net N$103: LED25.C, R102.2, R96.1, T48.C
- removed net N$104: LED25.A, R97.1
- removed net N$105: R98.1, T48.B
- removed net N$106: R99.1, T49.B
- removed net N$107: LED26.C, R100.1, R24.2, T50.C
- removed net N$108: LED26.A, R101.1
- removed net N$109: R102.1, T50.B
- removed net N$110: R105.1, T51.B
- removed net N$111: R106.2, T52.B
- removed net N$112: LED27.C, R104.1, R109.2, T51.C, T52.C
- removed net N$113: LED27.A, R103.1
- removed net N$114: LED28.C, R107.1, R112.2, T53.C
- removed net N$115: LED28.A, R108.1
- removed net N$116: R109.1, T53.B
- removed net N$117: T54.E, T55.C
- removed net N$118: LED29.C, R110.1, R116.2, T54.C
- removed net N$119: LED29.A, R111.1
- removed net N$120: R112.1, T54.B
- removed net N$121: R113.1, T55.B
- removed net N$122: LED30.C, R114.1, R26.2, T56.C
- removed net N$123: LED30.A, R115.1
- removed net N$124: R116.1, T56.B
- removed net N$125: T57.E, T58.C
- removed net N$126: LED31.C, R117.1, R123.2, T57.C
- removed net N$127: LED31.A, R118.1
- removed net N$128: R119.1, T57.B
- removed net N$129: R120.1, T58.B
- removed net N$130: LED32.C, R121.1, R125.2, T59.C
- removed net N$131: LED32.A, R122.1
- removed net N$132: R123.1, T59.B
- removed net N$133: R125.1, T60.B
- removed net N$134: R126.1, T61.B
- removed net N$135: R127.1, T62.B
- removed net N$136: R128.1, T63.B
- removed net N$137: LED33.C, R124.1, R132.2, T60.C, T61.C, T62.C, T63.C
- removed net N$138: LED33.A, R129.2
- removed net N$140: LED34.A, R131.1
- removed net N$141: R132.1, T64.B
- removed net N$142: R135.1, T65.B
- removed net N$143: R136.2, T66.B
- removed net N$144: LED35.C, R134.1, R139.2, T65.C, T66.C
- removed net N$145: LED35.A, R133.1
- removed net N$146: LED36.C, R137.1, R142.2, T67.C
- removed net N$147: LED36.A, R138.1
- removed net N$148: R139.1, T67.B
- removed net N$149: T68.E, T69.C
- removed net N$150: LED37.C, R140.1, R146.2, T68.C
- removed net N$151: LED37.A, R141.1
- removed net N$152: R142.1, T68.B
- removed net N$153: R143.1, T69.B
- removed net N$154: LED38.C, R128.2, R144.1, T70.C
- removed net N$155: LED38.A, R145.1
- removed net N$156: R146.1, T70.B
- removed net N$62: LED14.A, R58.1
- removed net N$65: LED15.C, R60.1, R66.2, T32.C
- removed net N$69: LED16.C, R126.2, R64.1, R85.2, T34.C
- removed net N$71: R66.1, T34.B
- removed net N$72: LED17.C, R67.1, R86.2, T35.C
- removed net N$73: LED17.A, R68.1
- removed net N$74: R69.1, T35.B
- removed net N$75: R72.1, T36.B
- removed net N$76: R73.2, T37.B
- removed net N$77: LED18.C, R71.1, R76.2, T36.C, T37.C
- removed net N$78: LED18.A, R70.1
- removed net N$79: LED19.C, R74.1, R79.2, T38.C
- removed net N$80: LED19.A, R75.1
- removed net N$81: R76.1, T38.B
- removed net N$82: T39.E, T40.C
- removed net N$83: LED20.C, R77.1, R83.2, T39.C
- removed net N$84: LED20.A, R78.1
- removed net N$85: R79.1, T39.B
- removed net N$86: R80.1, T40.B
- removed net N$88: LED21.A, R82.1
- removed net N$89: R83.1, T41.B
- removed net N$90: R85.1, T42.B
- removed net N$91: R86.1, T43.B
- removed net N$92: R87.1, T44.B
- removed net N$93: R88.1, T45.B
- removed net N$94: LED22.C, R84.1, R92.2, T42.C, T43.C, T44.C, T45.C
- removed net N$95: LED22.A, R89.2
- removed net N$97: LED23.A, R91.1
- removed net N$98: R92.1, T46.B
- new net N$41: R26.1, R48.2
- new net N$52: R27.1
- net !T: no longer R113.2, R143.2, R80.2
- net !Y: no longer R35.2, R62.2, R72.2
- net !Z: no longer R105.2, R120.2, R21.2, R54.2, R99.2
- net A: no longer LED9.C, R38.1, T22.C
- net B: no longer LED12.C, R48.1, T26.C
- net C: no longer LED14.C, R57.1, T31.C
- net D: no longer LED23.C, R90.1, T46.C
- net E: no longer LED21.C, R81.1, R87.2, T41.C
- net F: no longer LED24.C, R93.1, T47.C
- net G: no longer LED34.C, R130.1, T64.C
- net GND: now also T10.E, T11.E, T23.E, T8.E; no longer T13.E, T24.E, T26.E, T27.E, T28.E, T29.E, T3.E, T30.E, T31.E, T33.E, T34.E, T35.E, T36.E, T37.E, T38.E, T40.E, T41.E, T42.E, T43.E, T44.E, T45.E, T46.E, T47.E, T49.E, T50.E, T51.E, T52.E, T53.E, T55.E, T56.E, T58.E, T59.E, T60.E, T61.E, T62.E, T63.E, T64.E, T65.E, T66.E, T67.E, T69.E, T70.E
- net N$1: now also LED2.A, R14.1; no longer T8.E, T9.C
- net N$10: now also R8.2, T7.B; no longer R14.1, T3.B
- net N$11: now also R9.2, T8.B; no longer LED4.C, R14.2, R5.1, T8.C
- net N$12: now also R10.2, T9.B; no longer R15.1, T8.B
- net N$13: now also LED1.A, R12.1; no longer R16.1, T9.B
- net N$14: now also LED1.C, R11.1, R6.1, T1.C, T2.C; no longer R17.1, T4.B
- net N$15: now also R2.1, R24.2; no longer R18.1, T5.B
- net N$16: now also R1.1; no longer R19.1, T6.B
- net N$17: now also LED3.A, R16.1; no longer R20.1, T7.B
- net N$18: now also LED3.C, R15.1, R7.1, T6.C, T7.C, T8.C, T9.C; no longer LED3.A, R8.2
- net N$19: now also LED4.A, R18.1; no longer R22.1, T12.B
- net N$2: now also R13.1, R4.1; no longer R18.2, R3.1
- net N$20: now also LED4.C, R17.1, R21.1, T5.C; no longer T10.E, T11.C
- net N$21: now also LED5.A, R20.1; no longer LED5.C, R69.2, R9.1, T10.C
- net N$22: now also LED5.C, R19.1, T10.C; no longer LED5.A, R10.1
- net N$23: now also T3.E, T4.C; no longer R11.1, T10.B
- net N$24: now also R21.2, R8.1; no longer R21.1, T11.B
- net N$25: now also R3.1; no longer T11.E, T12.C
- net N$26: now also R5.1; no longer R24.1, T13.B
- net N$27: now also R25.2, T11.B; no longer R25.1, T14.B
- net N$28: now also R26.2, T12.B; no longer R26.1, T15.B
- net N$29: now also R22.2, R9.1; no longer R30.1, T16.B
- net N$3: now also R1.2; no longer R12.1
- net N$30: now also R10.1, R23.2; no longer LED6.C, R23.1, R95.2, T13.C, T14.C, T15.C
- net N$31: now also R27.2, T13.B; no longer LED6.A, R28.2
- net N$32: now also R28.2, T15.B; no longer R31.2, T17.B
- net N$33: now also R29.2, T14.B; no longer LED7.C, R29.1, R33.2, T16.C, T17.C
- net N$34: now also R30.2, T16.B; no longer LED7.A, R27.1
- net N$35: now also R31.2, T20.B; no longer R33.1, T18.B
- net N$36: now also R32.2, T17.B; no longer R34.1, T19.B
- net N$37: now also R33.2, T18.B; no longer R35.1, T20.B
- net N$38: now also R34.2, T19.B; no longer R36.1, T21.B
- net N$39: now also LED6.A, R36.1; no longer LED8.C, R32.1, R50.2, T18.C, T19.C, T20.C, T21.C
- net N$4: now also R2.2; no longer R13.2
- net N$40: now also LED6.C, R30.1, R35.1, T11.C, T12.C; no longer LED8.A, R37.2
- net N$42: now also R25.1; no longer LED9.A, R39.1
- net N$43: now also LED7.A, R38.1; no longer R40.1, T22.B
- net N$44: now also LED7.C, R28.1, R37.1, T13.C; no longer T23.E, T24.C
- net N$45: now also LED8.A, R40.1; no longer LED10.C, R41.1, R47.2, T23.C
- net N$46: now also LED8.C, R31.1, R39.1, T16.C, T17.C, T18.C, T19.C; no longer LED10.A, R42.1
- net N$47: now also LED9.A, R42.1; no longer R43.1, T23.B
- net N$48: now also LED9.C, R41.1, R45.1, T15.C; no longer R44.1, T24.B
- net N$49: now also LED10.A, R44.1; no longer LED11.C, R34.2, R45.1, T25.C
- net N$5: now also R3.2, T3.B; no longer LED4.A, R6.1
- net N$50: now also LED10.C, R43.1, T20.C; no longer LED11.A, R46.1
- net N$51: now also T13.E, T14.C; no longer R47.1, T25.B
- net N$53: now also R29.1; no longer LED12.A, R49.1
- net N$54: now also R33.1, R46.2; no longer R50.1, T26.B
- net N$55: now also R34.1, R47.2; no longer R52.1, T27.B
- net N$56: now also R32.1, R45.2; no longer R53.1, T28.B
- net N$57: now also R49.2, T21.B; no longer R54.1, T29.B
- net N$58: now also R50.2, T25.B; no longer R55.1, T30.B
- net N$59: now also R51.2, T22.B; no longer LED13.C, R51.1, R59.2, T27.C, T28.C, T29.C, T30.C
- net N$6: now also R4.2, T5.B; no longer LED1.C, R17.2, R2.1, T1.C, T2.C
- net N$60: now also R52.2, T23.B; no longer LED13.A, R56.2
- net N$63: now also LED11.A, R55.1; no longer R59.1, T31.B
- net N$64: now also LED11.C, R50.1, R54.1, T21.C, T22.C, T23.C; no longer T32.E, T33.C
- net N$66: now also LED12.A, R57.1; no longer LED15.A, R61.1
- net N$67: now also LED12.C, R56.1, T25.C; no longer R62.1, T32.B
- net N$68: now also R52.1, R59.2; no longer R63.1, T33.B
- net N$7: now also R5.2, T4.B; no longer LED1.A, R1.1
- net N$70: now also R51.1, R58.2; no longer LED16.A, R65.1
- net N$8: now also R6.2, T6.B; no longer LED2.A, R4.1
- net N$9: now also R7.2, T10.B; no longer LED3.C, R40.2, R7.1, T4.C, T5.C, T6.C, T7.C
- net T: no longer R13.1, R16.2, R22.2, R31.1, R44.2, R55.2
- net VCC: now also R11.2, R12.2, R13.2, R14.2, R15.2, R16.2, R17.2, R18.2, R19.2, R20.2, R35.2, R36.2, R37.2, R40.2, R43.2, R44.2, R54.2, R55.2, R56.2; no longer R1.2, R10.2, R100.2, R101.2, R103.2, R104.2, R107.2, R108.2, R110.2, R111.2, R114.2, R115.2, R117.2, R118.2, R121.2, R122.2, R124.2, R129.1, R130.2, R131.2, R133.2, R134.2, R137.2, R138.2, R140.2, R141.2, R144.2, R145.2, R2.2, R23.2, R27.2, R28.1, R29.2, R3.2, R32.2, R37.1, R4.2, R45.2, R46.2, R48.2, R49.2, R5.2, R51.2, R56.1, R58.2, R6.2, R60.2, R61.2, R64.2, R65.2, R67.2, R68.2, R7.2, R70.2, R71.2, R74.2, R75.2, R77.2, R78.2, R8.1, R81.2, R82.2, R84.2, R89.1, R9.2, R90.2, R91.2, R93.2, R94.2, R96.2, R97.2
- net X: no longer R127.2, R19.2, R25.2, R36.2, R52.2, R88.2
- net Y: no longer R106.1, R11.2, R119.2, R12.2, R135.2, R15.2, R53.2, R98.2
- net Z: no longer R136.1, R20.2, R30.2, R43.2, R63.2, R73.1
Other:
- moved on the sheet: LED1, LED10, LED11, LED12, LED2, LED3, LED4, LED5, LED6, LED7, LED8, LED9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

Commit message: final schema
Parts:
- removed R34: 10k, resistor:R-EU_M0805
- removed R47: (no value), rcl:R-EU_M1206
- removed T19: BC847, transistor-neu-to92:BC847
- added LED13, LED14, LED15, LED16, LED17, LED18, LED19, LED20, LED21, LED22, LED23, LED24, LED25, LED26, LED27, LED28, LED29, LED30, LED31, LED32, LED33, LED34: (no value), led:LEDCHIP-LED0805
- added R100, R107, R109, R115, R117, R122, R126, R131, R133, R139, R141, R149, R151, R65, R67, R75, R77, R82, R84, R89, R93, R98: (no value), resistor:R-EU_M0805
- added R101, R102, R103, R104, R105, R111, R113, R118, R119, R120, R124, R127, R128, R129, R134, R135, R136, R137, R145, R146, R147, R53, R60, R61, R62, R63, R71, R72, R73, R78, R79, R80, R85, R86, R87, R91, R94, R95, R96: 10k, resistor:R-EU_M0805
- added R106, R108, R114, R116, R121, R125, R130, R132, R138, R140, R148, R150, R64, R66, R74, R76, R81, R83, R88, R92, R97, R99: 3K9, resistor:R-EU_M0805
- added R110, R112, R123, R142, R143, R144, R68, R69, R70, R90: (no value), rcl:R-EU_M1206
- added T24, T26, T27, T28, T29, T30, T31, T32, T33, T34, T35, T36, T37, T38, T39, T40, T41, T42, T43, T44, T45, T46, T47, T48, T49, T50, T51, T52, T53, T54, T55, T56, T57, T58, T59, T60, T61, T62, T63: BC847, transistor-neu-to92:BC847
Connections:
- removed net N$16: R1.1
- removed net N$22: LED5.C, R19.1, T10.C
- removed net N$25: R3.1
- removed net N$26: R5.1
- removed net N$38: R34.2, T19.B
- removed net N$42: R25.1
- removed net N$50: LED10.C, R43.1, T20.C
- removed net N$52: R27.1
- removed net N$53: R29.1
- removed net N$55: R34.1, R47.2
- removed net N$67: LED12.C, R56.1, T25.C
- new net G_IN1: LED16.C, R118.1, R53.1, R76.1, T32.C
- new net G_IN2: LED26.C, R101.1, R116.1, R142.1, T49.C
- new net N$100: LED23.A, R107.1
- new net N$101: R86.2, T37.B
- new net N$102: R87.2, T38.B
- new net N$103: LED19.A, R89.1
- new net N$104: LED19.C, R88.1, R91.1, T37.C, T38.C
- new net N$105: LED23.C, R102.1, R106.1, T43.C, T44.C, T46.C
- new net N$106: LED24.A, R109.1
- new net N$107: R91.2, T39.B
- new net N$108: R94.2, T40.B
- new net N$109: LED20.A, R93.1
- new net N$111: R95.2, T42.B
- new net N$114: R105.1, R112.2
- new net N$115: R103.1, R110.2
- new net N$118: R113.2, T48.B
- new net N$119: LED17.C, R79.1, R81.1, T33.C
- new net N$121: LED25.A, R115.1
- new net N$125: T45.E, T48.C
- new net N$127: R96.2, T41.B
- new net N$129: LED21.C, R95.1, R97.1, T40.C
- new net N$132: R119.2, T50.B
- new net N$139: R87.1, R90.2
- new net N$141: R124.2, T52.B
- new net N$143: R127.2, T53.B
- new net N$144: LED20.C, R92.1, R94.1, T39.C
- new net N$145: T40.E, T41.C
- new net N$147: LED21.A, R98.1
- new net N$148: R128.2, T55.B
- new net N$151: LED29.C, R128.1, R130.1, T53.C
- new net N$152: T53.E, T54.C
- new net N$153: LED28.C, R125.1, R127.1, T52.C
- new net N$157: R134.2, T60.B
- new net N$158: R135.2, T57.B
- new net N$159: R136.2, T58.B
- new net N$160: R137.2, T59.B
- new net N$162: R136.1, R143.2
- new net N$164: R135.1, R142.2
- new net N$166: R137.1, R144.2
- new net N$168: R146.2, T63.B
- new net N$169: R147.2, T62.B
- new net N$173: T61.E, T62.C
- new net N$200: R71.2, T30.B
- new net N$251: LED27.A, R122.1
- new net N$252: LED27.C, R121.1, R124.1, T50.C, T51.C
- new net N$253: LED28.A, R126.1
- new net N$254: LED29.A, R131.1
- new net N$255: LED30.C, R112.1, R132.1, T55.C
- new net N$256: LED31.A, R139.1
- new net N$257: LED31.C, R134.1, R138.1, T56.C, T57.C, T58.C, T59.C
- new net N$258: LED32.A, R141.1
- new net N$260: LED33.A, R149.1
- new net N$261: LED33.C, R146.1, R148.1, T61.C
- new net N$262: LED34.C, R144.1, R150.1, T63.C
- new net N$263: R102.2, T47.B
- new net N$264: R104.2, T45.B
- new net N$265: R105.2, T46.B
- new net N$266: LED25.C, R111.1, R114.1, T45.C
- new net N$267: R111.2, T49.B
- new net N$269: R118.2, T56.B
- new net N$271: R120.1, R123.2
- new net N$272: R120.2, T51.B
- new net N$274: R129.2, T54.B
- new net N$61: R53.2, T24.B
- new net N$62: R60.2, T29.B
- new net N$65: R61.2, T26.B
- new net N$69: R62.2, T27.B
- new net N$71: R63.2, T28.B
- new net N$73: LED13.A, R65.1
- new net N$74: LED13.C, R60.1, R64.1, T24.C, T26.C, T27.C, T28.C
- new net N$75: R78.2, T33.B
- new net N$76: LED14.A, R67.1
- new net N$78: R62.1, R69.2
- new net N$79: R63.1, R70.2
- new net N$80: R61.1, R68.2
- new net N$81: T34.E, T36.C
- new net N$82: R72.2, T32.B
- new net N$83: R73.2, T31.B
- new net N$84: LED15.A, R75.1
- new net N$85: LED15.C, R72.1, R74.1, T30.C
- new net N$86: LED16.A, R77.1
- new net N$87: R79.2, T35.B
- new net N$88: T30.E, T31.C
- new net N$89: R101.2, T43.B
- new net N$91: R80.2, T34.B
- new net N$92: LED17.A, R82.1
- new net N$93: R103.2, T44.B
- new net N$94: LED18.A, R84.1
- new net N$95: T33.E, T34.C
- new net N$96: R145.2, T61.B
- new net N$98: LED18.C, R68.1, R83.1, T35.C
- new net N$99: R85.2, T36.B
- new net S$2: LED22.A, R100.1
- new net S$4: LED26.A, R117.1
- new net S$40: LED30.A, R133.1
- new net S$5: LED34.A, R151.1
- net !T: now also R129.1, R147.1, R96.1
- net !Y: now also R46.1, R71.1, R86.1
- net !Z: now also R113.1, R123.1, R59.1
- net A: now also LED5.C, R19.1, T10.C
- net B: now also LED10.C, R43.1, T20.C
- net C: now also LED12.C, R56.1, T25.C
- net D: now also LED14.C, R66.1, T29.C
- net E: now also LED22.C, R70.1, R99.1, T42.C
- net F: now also LED24.C, R108.1, T47.C
- net G: now also LED32.C, R140.1, T60.C
- net GND: now also T24.E, T26.E, T27.E, T28.E, T29.E, T31.E, T32.E, T35.E, T36.E, T37.E, T38.E, T39.E, T41.E, T42.E, T43.E, T44.E, T46.E, T47.E, T48.E, T49.E, T50.E, T51.E, T52.E, T54.E, T55.E, T56.E, T57.E, T58.E, T59.E, T60.E, T62.E, T63.E; no longer T19.E
- net N$46: no longer T19.C
- net T: now also R24.1, R29.1, R48.1, R5.1, R58.1, R80.1
- net VCC: now also R100.2, R106.2, R107.2, R108.2, R109.2, R114.2, R115.2, R116.2, R117.2, R121.2, R122.2, R125.2, R126.2, R130.2, R131.2, R132.2, R133.2, R138.2, R139.2, R140.2, R141.2, R148.2, R149.2, R150.2, R151.2, R64.2, R65.2, R66.2, R67.2, R74.2, R75.2, R76.2, R77.2, R81.2, R82.2, R83.2, R84.2, R88.2, R89.2, R92.2, R93.2, R97.2, R98.2, R99.2
- net X: now also R110.1, R143.1, R22.1, R69.1
- net Y: now also R1.1, R104.1, R119.1, R145.1, R3.1, R49.1, R78.1
- net Z: now also R23.1, R25.1, R27.1, R73.1, R85.1, R90.1

Commit message: final version of 2_10Decoder
Parts:
- removed T63: BC847, transistor-neu-to92:BC847
- added R152, R153, R154, R162, R163, R164, R165, R166, R167, R168, R169, R170, R171, R172, R173, R174, R175, R176, R177, R178, R179, R180, R181, R182, R183, R184, R185, R186, R187, R188, R189, R190, R191, R192, R193, R194, R195, R196, R197, R198, R199, R200, R201, R202, R203, R204, R205, R206, R207, R208, R209, R210, R211, R212, R213, R214, R215, R216, R217, R218, R219, R220, R221, R222, R223, R224, R225, R226, R227, R228, R229, R230, R231, R232, R233, R234, R235, R236, R237, R238, R239, R240, R241, R242, R243, R244, R245, R246, R247: (no value), rcl:R-EU_M1206
- added R155, R157, R47: 3K9, resistor:R-EU_M0805
- added R156, R158: (no value), resistor:R-EU_M0805
- added R159, R160, R161, R34: 10k, resistor:R-EU_M0805
- added T19: BC847, transistor-neu-to92:BC847
- JP1: SPICEPREFIX X -> (none)
- R1, R111, R113, R129, R134, R145, R25, R29, R31, R49, R5, R60, R63, R7, R71, R91, R94, R96: value 10k -> 3K9
- R100, R12, R122, R131, R139, R14, R149, R151, R36, R44, R67, R93, R98: value (none) -> 10k
- R102, R103, R105, R127, R128, R33, R62, R9: value 10k -> (none); device resistor:R-EU_M0805 -> rcl:R-EU_M1206
- R106, R140, R19, R43, R56, R83: value 3K9 -> (none); device resistor:R-EU_M0805 -> rcl:R-EU_M1206
- R107, R115, R141, R20, R42, R55, R57, R65, R82, R84: device resistor:R-EU_M0805 -> rcl:R-EU_M1206
- R11, R121, R13, R138, R148, R150, R35, R37, R54, R66, R81, R88, R99: value 3K9 -> 10k
- R112, R144, R48, R69, R90: device rcl:R-EU_M1206 -> resistor:R-EU_M0805
- R114, R130, R39, R41, R64, R92, R97: value 3K9 -> (none)
- R123, R142, R22, R23, R24, R45, R46, R70: value (none) -> 10k; device rcl:R-EU_M1206 -> resistor:R-EU_M0805
- R135, R146, R2, R26, R30, R32, R50, R6, R61, R72, R8, R95: value 10k -> (none)
- R143, R68: value (none) -> 3K9; device rcl:R-EU_M1206 -> resistor:R-EU_M0805
- R38, R40, R89: value (none) -> 3K9
Connections:
- new net N$110: R175.2, R176.1
- new net N$112: R178.2, R179.1
- new net N$113: R181.2, R182.1
- new net N$116: R185.2, R186.1
- new net N$117: R191.2, R192.1
- new net N$120: R194.2, R195.1
- new net N$122: R196.2, R197.1
- new net N$123: R198.2, R199.1
- new net N$124: R238.2, R239.1
- new net N$126: R241.2, R242.1
- new net N$128: R244.2, R245.1
- new net N$16: R103.2, R104.1
- new net N$22: R141.2, R142.1
- new net N$25: R106.2, R107.2
- new net N$26: R110.1, R115.1
- new net N$38: R105.2, R106.1
- new net N$42: R107.1, R110.2
- new net N$50: R62.1, R65.1
- new net N$52: R59.2, R62.2
- new net N$53: R58.1, R59.1
- new net N$55: R57.2, R58.2
- new net N$67: R162.2, R163.1
- new net N$72: R164.2, R165.1
- new net N$77: R167.2, R168.1
- new net N$90: R171.2, R172.1
- new net N$97: R173.2, R174.1
- new net S$123: LED24.C, R111.1, R115.2, R122.1, T43.C
- new net S$124: LED14.C, R63.1, R65.2, R78.1, T25.C
- net !T: now also R103.1, R141.1, R161.1, R229.1, R229.2, R230.1, R230.2, R231.1, R231.2, R236.1, R236.2, R237.1, R237.2; no longer R129.1, R147.1, R96.1
- net !Y: now also R190.1, R190.2, R200.1, R200.2, R226.1, R226.2, R227.1, R227.2, R228.1, R228.2, R42.1, R66.1, R98.1; no longer R46.1, R71.1, R86.1
- net !Z: now also R121.1, R140.1, R232.1, R232.2, R233.1, R233.2, R234.1, R234.2, R235.1, R235.2, R55.1, R88.1; no longer R113.1, R123.1, R59.1
- net A: now also JP1.17, LED2.C, R5.1, T3.C; no longer JP1.11, LED5.C, R19.1, T10.C
- net B: now also JP1.16, LED7.C, R29.1, T13.C; no longer JP1.12, LED10.C, R43.1, T20.C
- net C: now also JP1.15, LED11.C, R47.1, T20.C; no longer JP1.13, LED12.C, R56.1, T25.C
- net D: now also LED15.C, R68.1, T27.C; no longer LED14.C, R66.1, T29.C
- net E: now also JP1.13, R84.1, R96.1, T40.C; no longer JP1.15, R70.1, R99.1, T42.C
- net F: now also JP1.12, LED25.C, R113.1, T44.C; no longer JP1.16, LED24.C, R108.1, T47.C
- net G: now also JP1.11, LED31.C, R143.1, T55.C; no longer JP1.17, LED32.C, R140.1, T60.C
- net GND: now also R162.1, R163.2, R188.1, R188.2, R189.1, R189.2, R221.1, R221.2, R222.1, R222.2, R223.1, R223.2, R224.1, R224.2, R225.1, R225.2, T13.E, T19.E, T3.E, T30.E, T33.E, T40.E, T45.E, T53.E, T61.E; no longer T17.E, T24.E, T32.E, T39.E, T42.E, T52.E, T60.E, T63.E, T8.E
- net G_IN1: now also R153.1, R57.1; no longer LED16.C, R118.1, R53.1, R76.1, T32.C
- net G_IN2: now also R105.1, R154.1; no longer LED26.C, R101.1, R116.1, R142.1, T49.C
- net N$1: now also LED4.A, R16.1; no longer LED2.A, R14.1
- net N$10: now also R12.2, T5.B; no longer R8.2, T7.B
- net N$100: now also LED26.A, R117.1; no longer LED23.A, R107.1
- net N$101: now also R98.2; no longer R86.2
- net N$102: now also R99.2; no longer R87.2
- net N$103: now also LED20.A, R92.1; no longer LED19.A, R89.1
- net N$104: now also LED20.C, R93.1; no longer LED19.C, R88.1
- net N$105: now also LED26.C, R116.1, R120.1, T47.C, T48.C; no longer LED23.C, R102.1, R106.1, T43.C, T44.C
- net N$106: now also LED25.A, R114.1; no longer LED24.A, R109.1
- net N$107: now also R93.2, T36.B; no longer R91.2, T39.B
- net N$108: now also R100.2, T39.B; no longer R94.2, T40.B
- net N$109: now also LED19.A, R90.1; no longer LED20.A, R93.1
- net N$11: now also R13.2, T6.B; no longer R9.2, T8.B
- net N$111: now also R101.2, T40.B; no longer R95.2, T42.B
- net N$114: now also R124.1, R128.2; no longer R105.1, R112.2
- net N$115: now also R123.1, R127.2; no longer R103.1, R110.2
- net N$118: now also R121.2, T45.B; no longer R113.2, T48.B
- net N$119: now also R74.1, R86.1, T32.C; no longer R79.1, R81.1, T33.C
- net N$12: now also R14.2, T7.B; no longer R10.2, T9.B
- net N$121: now also LED23.A, R109.1; no longer LED25.A, R115.1
- net N$125: now also T42.E, T45.C; no longer T45.E, T48.C
- net N$127: now also R104.2; no longer R96.2
- net N$129: now also R101.1, R94.1, T39.C; no longer R95.1, R97.1, T40.C
- net N$13: now also R2.1; no longer R12.1
- net N$132: now also R136.2; no longer R119.2
- net N$139: now also R102.2, R99.1; no longer R87.1, R90.2
- net N$14: now also R1.1; no longer R6.1
- net N$141: now also R131.2, T49.B; no longer R124.2, T52.B
- net N$143: now also R138.2, T52.B; no longer R127.2, T53.B
- net N$144: now also LED19.C, R100.1, R89.1, T36.C; no longer LED20.C, R92.1, R94.1, T39.C
- net N$145: now also T39.E; no longer T40.E
- net N$147: now also R95.1; no longer R98.1
- net N$148: now also R139.2, T53.B; no longer R128.2, T55.B
- net N$15: now also R4.1, R9.2; no longer R2.1, R24.2
- net N$151: now also R132.1, R139.1, T52.C; no longer R128.1, R130.1, T53.C
- net N$152: now also T52.E; no longer T53.E
- net N$153: now also LED27.C, R138.1, T49.C; no longer LED28.C, R127.1, T52.C
- net N$157: now also R147.2, T55.B; no longer R134.2, T60.B
- net N$158: now also R149.2; no longer R135.2
- net N$159: now also R150.2; no longer R136.2
- net N$160: now also R151.2; no longer R137.2
- net N$162: now also R150.1, R153.2; no longer R136.1, R143.2
- net N$164: now also R149.1, R152.2; no longer R135.1, R142.2
- net N$166: now also R151.1, R154.2; no longer R137.1, R144.2
- net N$168: now also R160.2, T61.B; no longer R146.2, T63.B
- net N$169: now also R161.2; no longer R147.2
- net N$17: now also R8.1; no longer R16.1
- net N$173: now also T60.E; no longer T61.E
- net N$18: now also R10.1, T4.C, T5.C; no longer R15.1, T8.C, T9.C
- net N$19: now also LED5.A; no longer LED4.A
- net N$2: now also LED4.C, R15.1, R23.1, T8.C; no longer LED2.C, R13.1, R4.1, T3.C
- net N$20: now also LED5.C, T9.C; no longer LED4.C, T5.C
- net N$200: now also R66.2, T24.B; no longer R71.2, T30.B
- net N$21: now also LED2.A, R6.1; no longer LED5.A, R20.1
- net N$23: now also T10.C, T8.E; no longer T3.E, T4.C
- net N$24: now also R12.1; no longer R8.1
- net N$251: now also LED28.A, R130.1; no longer LED27.A, R122.1
- net N$252: now also LED28.C, R129.1, R131.1; no longer LED27.C, R121.1, R124.1
- net N$253: now also LED27.A; no longer LED28.A
- net N$254: now also R133.1; no longer R131.1
- net N$255: now also R128.1, R134.1, T53.C; no longer R112.1, R132.1, T55.C
- net N$256: now also LED32.A, R146.1; no longer LED31.A, R139.1
- net N$257: now also LED32.C, R145.1, R147.1; no longer LED31.C, R134.1, R138.1
- net N$258: now also LED31.A, R144.1; no longer LED32.A, R141.1
- net N$260: now also R156.1; no longer R149.1
- net N$261: now also R155.1, R160.1, T60.C; no longer R146.1, R148.1, T61.C
- net N$262: now also R152.1, R157.1, T61.C; no longer R144.1, R150.1, T63.C
- net N$263: now also R120.2, T44.B; no longer R102.2, T47.B
- net N$264: now also R118.2, T42.B; no longer R104.2, T45.B
- net N$265: now also R124.2, T48.B; no longer R105.2, T46.B
- net N$266: now also LED23.C, R108.1, R119.1, T42.C; no longer LED25.C, R111.1, R114.1, T45.C
- net N$267: now also R119.2, T43.B; no longer R111.2, T49.B
- net N$269: now also R148.2; no longer R118.2
- net N$27: now also R27.2; no longer R25.2
- net N$271: now also R137.1, R140.2; no longer R120.1, R123.2
- net N$272: now also R137.2; no longer R120.2
- net N$274: now also R142.2; no longer R129.2
- net N$28: now also R28.2; no longer R26.2
- net N$29: now also R13.1, R19.2; no longer R22.2, R9.1
- net N$3: now also R3.2; no longer R1.2
- net N$30: now also R14.1, R20.2; no longer R10.1, R23.2
- net N$31: now also R44.2, T17.B; no longer R27.2, T13.B
- net N$32: now also R45.2, T18.B; no longer R28.2, T15.B
- net N$33: now also R46.2, T19.B; no longer R29.2, T14.B
- net N$34: now also R35.2, T14.B; no longer R30.2, T16.B
- net N$35: now also R34.2, T13.B; no longer R31.2, T20.B
- net N$36: now also R36.2, T15.B; no longer R32.2, T17.B
- net N$37: now also R37.2, T16.B; no longer R33.2, T18.B
- net N$39: now also R26.1; no longer R36.1
- net N$4: now also R4.2; no longer R2.2
- net N$40: now also R25.1; no longer R30.1
- net N$41: now also R28.1, R33.2; no longer R26.1, R48.2
- net N$43: now also LED9.A, R39.1; no longer LED7.A, R38.1
- net N$44: now also LED9.C, R38.1, R45.1, T17.C; no longer LED7.C, R28.1, R37.1, T13.C
- net N$45: now also R32.1; no longer R40.1
- net N$46: now also R34.1, T14.C, T15.C; no longer R39.1, T17.C, T18.C
- net N$47: now also LED10.A, R41.1; no longer LED9.A, R42.1
- net N$48: now also LED10.C, R40.1, R43.1, T18.C; no longer LED9.C, R41.1, R45.1, T15.C
- net N$49: now also LED7.A, R30.1; no longer LED10.A, R44.1
- net N$5: now also R22.2, T8.B; no longer R3.2, T3.B
- net N$51: now also T17.E, T19.C; no longer T13.E, T14.C
- net N$54: now also R37.1, R42.2; no longer R33.1, R46.2
- net N$56: now also R36.1, R43.2; no longer R32.1, R45.2
- net N$57: now also R52.2; no longer R49.2
- net N$58: now also R51.2, T20.B; no longer R50.2, T25.B
- net N$59: now also R53.2; no longer R51.2
- net N$6: now also R23.2, T9.B; no longer R4.2, T5.B
- net N$60: now also R54.2; no longer R52.2
- net N$61: now also R78.2, T28.B; no longer R53.2, T24.B
- net N$62: now also R73.2, T27.B; no longer R60.2, T29.B
- net N$63: now also LED12.A, R50.1; no longer LED11.A, R55.1
- net N$64: now also LED12.C, R49.1, R51.1; no longer LED11.C, R50.1, R54.1
- net N$65: now also R79.2, T29.B; no longer R61.2, T26.B
- net N$66: now also LED11.A, R48.1; no longer LED12.A, R57.1
- net N$68: now also R54.1, R55.2; no longer R52.1, R59.2
- net N$69: now also R80.2, T30.B; no longer R62.2, T27.B
- net N$7: now also R24.2, T10.B; no longer R5.2, T4.B
- net N$70: now also R53.1, R56.2; no longer R51.1, R58.2
- net N$71: now also R81.2, T31.B; no longer R63.2, T28.B
- net N$73: now also LED16.A, R72.1; no longer LED13.A, R65.1
- net N$74: now also LED16.C, R71.1, R73.1, T29.C, T30.C, T31.C; no longer LED13.C, R60.1, R64.1, T24.C, T26.C, T27.C
- net N$75: now also R85.2, T32.B; no longer R78.2, T33.B
- net N$76: now also LED15.A, R69.1; no longer LED14.A, R67.1
- net N$78: now also R80.1, R83.2; no longer R62.1, R69.2
- net N$79: now also R81.1, R84.2; no longer R63.1, R70.2
- net N$8: now also R11.2, T4.B; no longer R6.2, T6.B
- net N$80: now also R79.1, R82.2; no longer R61.1, R68.2
- net N$81: now also T35.C; no longer T36.C
- net N$82: now also R67.2, T25.B; no longer R72.2, T32.B
- net N$83: now also R70.2, T26.B; no longer R73.2, T31.B
- net N$84: now also LED13.A, R61.1; no longer LED15.A, R75.1
- net N$85: now also LED13.C, R60.1, R67.1, T24.C; no longer LED15.C, R72.1, R74.1, T30.C
- net N$86: now also LED14.A, R64.1; no longer LED16.A, R77.1
- net N$87: now also R86.2, T33.B; no longer R79.2, T35.B
- net N$88: now also T24.E, T26.C; no longer T30.E, T31.C
- net N$89: now also R122.2, T46.B; no longer R101.2, T43.B
- net N$9: now also R10.2, T3.B; no longer R7.2, T10.B
- net N$91: now also R87.2; no longer R80.2
- net N$92: now also R75.1; no longer R82.1
- net N$93: now also R123.2, T47.B; no longer R103.2, T44.B
- net N$94: now also R77.1; no longer R84.1
- net N$95: now also T32.E; no longer T33.E
- net N$96: now also R159.2, T60.B; no longer R145.2, T61.B
- net N$98: now also R76.1, R82.1, T33.C; no longer R68.1, R83.1, T35.C
- net N$99: now also R88.2, T35.B; no longer R85.2, T36.B
- net S$2: now also R97.1; no longer R100.1
- net S$4: now also LED24.A, R112.1; no longer LED26.A, R117.1
- net S$40: now also R135.1; no longer R133.1
- net S$5: now also R158.1; no longer R151.1
- net T: now also R184.1, R184.2, R215.1, R215.2, R216.1, R216.2, R33.1, R46.1, R56.1, R87.1, R9.1; no longer R29.1, R48.1, R5.1, R58.1, R80.1
- net VCC: now also R1.2, R111.2, R112.2, R113.2, R129.2, R134.2, R135.2, R143.2, R144.2, R145.2, R146.2, R155.2, R156.2, R157.2, R158.2, R164.1, R165.2, R171.1, R172.2, R173.1, R174.2, R175.1, R176.2, R178.1, R179.2, R180.1, R180.2, R182.2, R183.1, R185.1, R186.2, R187.1, R187.2, R194.1, R195.2, R196.1, R197.2, R198.1, R199.2, R2.2, R238.1, R239.2, R240.1, R240.2, R241.1, R242.2, R243.1, R243.2, R244.1, R245.2, R246.1, R246.2, R247.1, R247.2, R25.2, R26.2, R29.2, R30.2, R31.2, R32.2, R47.2, R48.2, R49.2, R5.2, R50.2, R6.2, R60.2, R61.2, R63.2, R68.2, R69.2, R7.2, R71.2, R72.2, R8.2, R90.2, R91.2, R94.2, R95.2, R96.2; no longer R100.2, R106.2, R107.2, R11.2, R115.2, R12.2, R121.2, R122.2, R13.2, R131.2, R138.2, R139.2, R14.2, R140.2, R141.2, R148.2, R149.2, R150.2, R151.2, R19.2, R20.2, R35.2, R36.2, R37.2, R42.2, R43.2, R44.2, R54.2, R55.2, R56.2, R57.2, R65.2, R66.2, R67.2, R81.2, R82.2, R83.2, R84.2, R88.2, R93.2, R98.2, R99.2
- net X: now also R127.1, R148.1, R167.1, R168.2, R19.1, R208.1, R208.2, R209.1, R209.2, R210.1, R210.2, R211.1, R211.2, R212.1, R212.2, R217.1, R217.2, R218.1, R218.2, R219.1, R219.2, R220.1, R220.2, R83.1; no longer R110.1, R143.1, R22.1, R69.1
- net Y: now also R118.1, R136.1, R159.1, R166.1, R166.2, R181.1, R183.2, R201.1, R201.2, R202.1, R202.2, R203.1, R203.2, R204.1, R204.2, R205.1, R205.2, R206.1, R206.2, R207.1, R207.2, R22.1, R52.1, R85.1; no longer R1.1, R104.1, R119.1, R145.1, R49.1, R78.1
- net Z: now also R102.1, R169.1, R169.2, R170.1, R170.2, R177.1, R177.2, R191.1, R192.2, R193.1, R193.2, R20.1, R213.1, R213.2, R214.1, R214.2, R44.1, R70.1; no longer R23.1, R25.1, R73.1, R85.1, R90.1
Other:
- moved on the sheet: JP1, LED10, LED11, LED12, LED13, LED14, LED15, LED16, LED19, LED2, LED20, LED23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
